File: Game Gear Breakout.kicad_pcb (KiCad board)
At the start: 2 copper layers, 12 parts, among them J1 GG Edge Connector, J2 Logic Analyzer, J3 ROM Chip

Commit message: bottom routed (try #1)
Parts:
- removed C2: 1u, Capacitor_SMD:C_0805_2012Metric_Pad1.18x1.45mm_HandSolder
- removed TP1, TP2: TestPoint, TestPoint:TestPoint_Pad_2.0x2.0mm
- added PEG1: MountingHole, MountingHole:MountingHole_2.7mm_M2.5, F.Cu at (128.1, 78.4)
- added PEG2: MountingHole, MountingHole:MountingHole_2.7mm_M2.5, F.Cu at (181.2, 104.8)
- R1, R2: moved to B.Cu
- moved D2 89.2 mm to (129.5, 68.7), turned to 90 degrees
- moved R2 79.5 mm to (129.4, 68.8), turned to 90 degrees
- moved R1 69.6 mm to (126.8, 68.7), turned to 90 degrees
- moved D1 66.4 mm to (126.8, 68.7), turned to 90 degrees
- moved C1 64.9 mm to (163.8, 85.5), turned to 90 degrees
- moved J2 62.9 mm to (126.7, 64.1), turned to 90 degrees
- moved JP1 57.3 mm to (177.2, 116.4)
- moved J3 47.1 mm to (154.6, 95.0)
- moved J1 0.30 mm to (154.5, 102.7)
Connections:
- J1 pad 41: GND -> /Pin 41
- J2 pad 46: unconnected-(J2-Pad46) -> GND
Routing:
- net +5V: track 0.00 -> 134.3 mm, vias 0 -> 2
- net /+34V: track 0.00 -> 77.9 mm, vias 0 -> 2
- net /~{WR}: track 0.00 -> 68.5 mm, vias 0 -> 1
- net /~{TV}: track 0.00 -> 68.2 mm, vias 0 -> 1
- net /TV_L: track 0.00 -> 67.4 mm, vias 0 -> 1
- net /~{IOReg}: track 0.00 -> 67.2 mm, vias 0 -> 1
- net /D2: track 0.00 -> 67.2 mm, vias 0 -> 1
- net /A5: track 0.00 -> 67.2 mm, vias 0 -> 1
- net /A11: track 0.00 -> 67.2 mm, vias 0 -> 1
- net /A8: track 0.00 -> 67.2 mm, vias 0 -> 1
- net /A3: track 0.00 -> 67.2 mm, vias 0 -> 1
- net /~{RESET}: track 0.00 -> 67.2 mm, vias 0 -> 1
- net /~{M0-7}: track 0.00 -> 67.2 mm, vias 0 -> 1
- net /Pin 41: track 0.00 -> 67.2 mm, vias 0 -> 1
- net /D7: track 0.00 -> 67.2 mm, vias 0 -> 1
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- added copper zone on B.Cu, net GND
- added copper zone on F.Cu, net GND
Other:
- board outline added: 59.1 x 73 mm

Commit message: rev1 layout done?
Parts:
- added REF**: OSHW-Symbol_6.7x6mm_SilkScreen, Symbol:OSHW-Symbol_6.7x6mm_SilkScreen, F.Cu at (145.0, 95.4)
- added REF**: KiCad-Logo2_5mm_SilkScreen, Symbol:KiCad-Logo2_5mm_SilkScreen, F.Cu at (162.7, 112.5)
- added TP1: TestPoint, My Libraries:Harwin-S1751-46-Test-Point, F.Cu at (165.9, 72.9)
- added TP2: TestPoint, My Libraries:Harwin-S1751-46-Test-Point, F.Cu at (183.8, 72.9)
- added TP3: TestPoint, My Libraries:Harwin-S1751-46-Test-Point, F.Cu at (145.4, 72.8)
- added TP4: TestPoint, My Libraries:Harwin-S1751-46-Test-Point, F.Cu at (179.2, 87.1)
- added kibuzzard-638A45B3: G***, kibuzzard-638A45B3, F.Cu at (137.4, 75.1)
- added kibuzzard-638A45B3: G***, kibuzzard-638A45B3, F.Cu at (179.1, 89.5)
- added kibuzzard-638A45BD: G***, kibuzzard-638A45BD, F.Cu at (134.8, 75.1)
- added kibuzzard-638A4743: G***, kibuzzard-638A4743, F.Cu at (189.0, 112.4)
- added kibuzzard-638A474E: G***, kibuzzard-638A474E, F.Cu at (183.1, 112.1)
- added kibuzzard-638A50E1: G***, kibuzzard-638A50E1, F.Cu at (162.7, 78.9)
- added svg2mod: G***, My Libraries:BE5v2, F.Cu at (180.5, 93.0)
- moved D1 10.6 mm to (137.3, 69.5)
- moved R1 10.6 mm to (137.4, 69.5)
- moved JP1 9.84 mm to (186.1, 112.1)
- moved C1 8.09 mm to (171.9, 85.9)
- moved J1 8.09 mm to (162.6, 103.2)
- moved J3 8.09 mm to (162.7, 95.4)
- moved PEG1 8.09 mm to (136.2, 78.8)
- moved PEG2 8.09 mm to (189.2, 105.2)
- moved J2 8.09 mm to (134.7, 64.5)
- moved R2 5.44 mm to (134.8, 69.5)
- moved D2 5.43 mm to (134.8, 69.5)
Routing:
- net /A7: track 67.2 -> 120.5 mm
- net /A12: track 65.8 -> 116.6 mm
- net /A5: track 67.2 -> 115.5 mm
- net /A14: track 67.2 -> 114.7 mm
- net +5V: track 134.3 -> 181.2 mm, vias 2 -> 4
- net /A6: track 65.2 -> 110.9 mm
- net /A8: track 67.2 -> 111.4 mm
- net /A3: track 67.2 -> 110.5 mm
- net /A11: track 67.2 -> 109.2 mm
- net /A4: track 65.2 -> 106.1 mm
- net /A13: track 65.2 -> 105.9 mm
- net /A10: track 67.2 -> 107.6 mm
- net /D7: track 67.2 -> 105.5 mm
- net /A1: track 67.2 -> 105.2 mm
- net /A9: track 65.2 -> 103.0 mm
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Other:
- board size 59.1 x 73 mm -> 59.1 x 73.5 mm
- board text added: "+34V"
- board text added: "+5V"
- board text added: "41"
- board text added: "5V"
- board text added: "A0"
- board text added: "A1"
- board text added: "A10"
- board text added: "A11"
- board text added: "A12"
- board text added: "A13"
- board text added: "A14"
- board text added: "A15"
- board text added: "A2"
- board text added: "A3"
- board text added: "A4"
- board text added: "A5"
- board text added: "A6"
- board text added: "A7"
- board text added: "A8"
- board text added: "A9"
- board text added: "Clk"
- board text added: "Clock"
- board text added: "D0"
- board text added: "D1"
- board text added: "D2"
- board text added: "D3"
- board text added: "D4"
- board text added: "D5"
- board text added: "D6"
- board text added: "D7"
- board text added: "Pin 41"
- board text added: "~{CE}"
- board text added: "~{GG}"
- board text added: "~{IOReq}"
- board text added: "~{IO}"
- board text added: "~{L}"
- board text added: "~{M0-7}"
- board text added: "~{M0}"
- board text added: "~{M1}"
- board text added: "~{M8-B}"
- board text added: "~{M8}"
- board text added: "~{RD}"
- board text added: "~{RESET}"
- board text added: "~{RES}"
- board text added: "~{Refresh}"
- board text added: "~{Rfh}"
- board text added: "~{R}"
- board text added: "~{TV_L}"
- board text added: "~{TV_R}"
- board text added: "~{TV}"
- board text added: "~{WR}"

Commit message: v1 submitting to fab
Parts:
- moved J2 5.08 mm to (134.7, 59.5)
- moved TP2 3.44 mm to (184.7, 69.6)
- moved TP3 3.44 mm to (146.2, 69.5)
- moved TP1 3.44 mm to (166.8, 69.6)
Routing:
- net +5V: track 181.2 -> 190.9 mm
- net /D1: track 91.9 -> 97.5 mm
- net /+34V: track 68.2 -> 73.3 mm
- net /~{RD}: track 101.5 -> 106.6 mm
- net /~{M8-B}: track 65.2 -> 70.3 mm
- net /~{M1}: track 65.2 -> 70.3 mm
- net /~{CE}: track 65.2 -> 70.3 mm
- net /Pin 41: track 84.4 -> 89.4 mm
- net /D4: track 93.2 -> 98.2 mm
- net /Clock: track 65.2 -> 70.3 mm
- net /A6: track 110.9 -> 116.0 mm
- net /A4: track 106.1 -> 111.1 mm
- net /A2: track 100.6 -> 105.6 mm
- net /A14: track 114.7 -> 119.7 mm
- net /A12: track 116.6 -> 121.7 mm
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Other:
- board size 59.1 x 73.5 mm -> 59.1 x 78.6 mm

Commit message: gerbs and pdf of schematic (v1)
Changed lines of the file:
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@@
       (outputformat 1)
       (mirror false)
-      (drillshape 1)
+      (drillshape 0)
       (scaleselection 1)
       (outputdirectory "")
@@
     (fp_line (start 1.6 -0.8) (end -1.2 -0.8) (layer "F.Fab") (width 0.1))
     (fp_line (start -1.6 0.8) (end 1.6 0.8) (layer "F.Fab") (width 0.1))
-    (pad "1" smd roundrect (at -1.4875 0 90) (size 1.425 1.75) (layers "F.Cu" "F.Paste" "F.Mask") (roundrect_rratio 0.175439)
+    (pad "1" smd roundrect (at -1.4875 0 90) (size 1.425 1.75) (layers "F.Cu" "F.Paste" "F.Mask") (roundrect_rratio 0.1754392982)
       (net 2 "GND") (pinfunction "K") (pintype "passive"))
-    (pad "2" smd roundrect (at 1.4875 0 90) (size 1.425 1.75) (layers "F.Cu" "F.Paste" "F.Mask") (roundrect_rratio 0.175439)
+    (pad "2" smd roundrect (at 1.4875 0 90) (size 1.425 1.75) (layers "F.Cu" "F.Paste" "F.Mask") (roundrect_rratio 0.1754392982)
       (net 3 "Net-(D1-Pad2)") (pinfunction "A") (pintype "passive"))
     (model "${KICAD6_3DMODEL_DIR}/LED_SMD.3dshapes/LED_1206_3216Metric.wrl"
@@
     (fp_line (start 1.6 -0.8) (end -1.2 -0.8) (layer "F.Fab") (width 0.1))
     (fp_line (start -1.2 -0.8) (end -1.6 -0.4) (layer "F.Fab") (width 0.1))
-    (pad "1" smd roundrect (at -1.4875 0 90) (size 1.425 1.75) (layers "F.Cu" "F.Paste" "F.Mask") (roundrect_rratio 0.175439)
+    (pad "1" smd roundrect (at -1.4875 0 90) (size 1.425 1.75) (layers "F.Cu" "F.Paste" "F.Mask") (roundrect_rratio 0.1754392982)
       (net 2 "GND") (pinfunction "K") (pintype "passive"))
-    (pad "2" smd roundrect (at 1.4875 0 90) (size 1.425 1.75) (layers "F.Cu" "F.Paste" "F.Mask") (roundrect_rratio 0.175439)
+    (pad "2" smd roundrect (at 1.4875 0 90) (size 1.425 1.75) (layers "F.Cu" "F.Paste" "F.Mask") (roundrect_rratio 0.1754392982)
       (net 4 "Net-(D2-Pad2)") (pinfunction "A") (pintype "passive"))
     (model "${KICAD6_3DMODEL_DIR}/LED_SMD.3dshapes/LED_1206_3216Metric.wrl"
@@
     (fp_line (start -1 -0.625) (end 1 -0.625) (layer "F.Fab") (width 0.1))
     (fp_line (start 1 -0.625) (end 1 0.625) (layer "F.Fab") (width 0.1))
-    (pad "1" smd roundrect (at -1.0375 0 90) (size 1.175 1.45) (layers "F.Cu" "F.Paste" "F.Mask") (roundrect_rratio 0.212766)
+    (pad "1" smd roundrect (at -1.0375 0 90) (size 1.175 1.45) (layers "F.Cu" "F.Paste" "F.Mask") (roundrect_rratio 0.2127659574)
       (net 1 "+5V") (pintype "passive"))
-    (pad "2" smd roundrect (at 1.0375 0 90) (size 1.175 1.45) (layers "F.Cu" "F.Paste" "F.Mask") (roundrect_rratio 0.212766)
+    (pad "2" smd roundrect (at 1.0375 0 90) (size 1.175 1.45) (layers "F.Cu" "F.Paste" "F.Mask") (roundrect_rratio 0.2127659574)
       (net 2 "GND") (pintype "passive"))
     (model "${KICAD6_3DMODEL_DIR}/Capacitor_SMD.3dshapes/C_0805_2012Metric.wrl"
@@
     (fp_line (start 1 0.625) (end 1 -0.625) (layer "B.Fab") (width 0.1))
     (fp_line (start 1 -0.625) (end -1 -0.625) (layer "B.Fab") (width 0.1))
-    (pad "1" smd roundrect (at -1 0 90) (size 1.2 1.4) (layers "B.Cu" "B.Paste" "B.Mask") (roundrect_rratio 0.208333)
+    (pad "1" smd roundrect (at -1 0 90) (size 1.2 1.4) (layers "B.Cu" "B.Paste" "B.Mask") (roundrect_rratio 0.2083333333)
       (net 5 "/+34V") (pintype "passive"))
-    (pad "2" smd roundrect (at 1 0 90) (size 1.2 1.4) (layers "B.Cu" "B.Paste" "B.Mask") (roundrect_rratio 0.208333)
+    (pad "2" smd roundrect (at 1 0 90) (size 1.2 1.4) (layers "B.Cu" "B.Paste" "B.Mask") (roundrect_rratio 0.2083333333)
       (net 4 "Net-(D2-Pad2)") (pintype "passive"))
     (model "${KICAD6_3DMODEL_DIR}/Resistor_SMD.3dshapes/R_0805_2012Metric.wrl"
@@
     (fp_line (start 1 0.625) (end 1 -0.625) (layer "B.Fab") (width 0.1))
     (fp_line (start -1 0.625) (end 1 0.625) (layer "B.Fab") (width 0.1))
-    (pad "1" smd roundrect (at -1 0 90) (size 1.2 1.4) (layers "B.Cu" "B.Paste" "B.Mask") (roundrect_rratio 0.208333)
+    (pad "1" smd roundrect (at -1 0 90) (size 1.2 1.4) (layers "B.Cu" "B.Paste" "B.Mask") (roundrect_rratio 0.2083333333)
       (net 1 "+5V") (pintype "passive"))
-    (pad "2" smd roundrect (at 1 0 90) (size 1.2 1.4) (layers "B.Cu" "B.Paste" "B.Mask") (roundrect_rratio 0.208333)
+    (pad "2" smd roundrect (at 1 0 90) (size 1.2 1.4) (layers "B.Cu" "B.Paste" "B.Mask") (roundrect_rratio 0.2083333333)
       (net 3 "Net-(D1-Pad2)") (pintype "passive"))
     (model "${KICAD6_3DMODEL_DIR}/Resistor_SMD.3dshapes/R_0805_2012Metric.wrl"
